File: hardware/imu.kicad_pcb (KiCad board)
At the start: 4 copper layers, 40 x 40 mm, 108 parts, among them J1 USB-MINI-B-SMD, J2 DRILL, J3 DRILL, J4 DRILL, J5 DRILL, J6 STACK-UP-LOW, J7 STACK-DOWN, J8 STACK-UP-LOW, J9 STACK-DOWN, P1 CON-SENSOR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

Commit message: Add new 3d model
Parts:
- FB401, FB402: footprint C0603 -> kicad-libraries:C0603
- FILTER401, FILTER402: footprint DFN16-33x135 -> kicad-libraries:DFN16-33x135
